File: Proyecto Parcticas.kicad_sch (KiCad schematic)
At the start: 8 parts

Commit message: Ultima versión
Parts:
- added BT1: Battery_Cell, Connector_Molex:Molex_KK-254_AE-6410-02A_1x02_P2.54mm_Vertical, symbol Device:Battery_Cell
- added C2: (no value), Capacitor_SMD:CP_Elec_5x5.4, symbol Device:C_Polarized
- added C3: 10uF, Capacitor_SMD:CP_Elec_5x5.4, symbol Device:C_Polarized
- added C4: (no value), symbol Device:C
- added J1: Bateria Lipo, TerminalBlock:TerminalBlock_bornier-2_P5.08mm, symbol Connector:Screw_Terminal_01x02
- added J2: Micro_SD_Card, symbol MicroSD:Micro_SD_Card
- added R? (x2): (no value), symbol Device:R
- added uC1: Esp32s, Esp32:Esp32, symbol ESP32s:Esp32s
- C1: renamed from C?; value (none) -> Modulo_de_Carga_USB-C; footprint (none) -> Modulo_de_carga_USB_C:Modulo_de_carga_USB_C
- DS1: renamed from DS?; footprint LCD_AOM12864A0-1.54WW-ANO -> Connector_Molex:Molex_KK-254_AE-6410-06A_1x06_P2.54mm_Vertical
- E1: renamed from E?; value (none) -> Encoder_rotativo; footprint (none) -> Connector_Molex:Molex_KK-254_AE-6410-05A_1x05_P2.54mm_Vertical
- F1: renamed from F?; value (none) -> StepUp 5v; footprint (none) -> StepUp:StepUp
- S1: renamed from S?; value (none) -> Sensor_Infrarrojo; footprint (none) -> Connector_Molex:Molex_KK-254_AE-6410-03A_1x03_P2.54mm_Vertical
- S2: renamed from S?; value (none) -> XH711; footprint (none) -> HX711:HX711
- S3: renamed from S?; value (none) -> Sensor_de_Carga; footprint (none) -> Connector_Molex:Molex_KK-254_AE-6410-04A_1x04_P2.54mm_Vertical
- U1: renamed from U?; value (none) -> Sensor_de_corriente_ACS758LCB
Connections:
- net BAT+: now reaches C1. (BT-)
- net BAT+: now also F1.1 (VIN+), BT1.1 (+), R?.1
- net at S3. (E-): now also S2.4 (E-)
- net VCC: now reaches S1. (VCC)
- net VCC: now also DS1.2 (VCC), E1. (SW), F1.3 (OUT+), S2.8 (VCC), U1. (VCC), J2.5 (VCC), uC1. (TX)
- net GND: now reaches DS1.1 (GND)
- net GND: now also E1. (SW), F1.4 (OUT-), S1. (VCC), S2.5 (GND), U1. (VCC), C2.2, C3.2, C4.2, J2.6 (GND), R?.2, uC1. (TX)
- net D_SCL: now reaches DS1.4 (SCL)
- net D_SCL: now also uC1. (TX)
- net D_DC: now reaches DS1.5 (DC)
- net D_DC: now also uC1. (TX)
- net D_RES: now reaches DS1.6 (RES)
- net D_RES: now also uC1. (TX)
- net D_SDA: now reaches DS1.7 (SDA)
- net D_SDA: now also uC1. (TX)
- new net: BT1.2 (-), C1. (BT-)
- new net: J1.1 (Pin_1), U1. (VCC)
- new net: J1.2 (Pin_2), U1. (VCC)
- new net: S2.1 (A+), S3. (E-)
- new net: S2.2 (A-), S3. (E-)
- new net: S2.3 (E+), S3. (E-)
- new net: C3.1, C4.1, uC1. (TX)
- new net BAT+_EXT: uC1. (TX)
- new net BAT+_INT: R?.1, R?.2, uC1. (TX)
- new net E_CLK: E1. (SW), uC1. (TX)
- new net E_DT: E1. (SW), uC1. (TX)
- new net E_SW: E1. (SW), uC1. (TX)
- new net PIN_BNT_STOP: uC1. (TX)
- new net PWM_OUT: uC1. (TX)
- new net SD_CS: J2.1 (CS), uC1. (TX)
- new net SD_MISO: J2.4 (MISO), uC1. (TX)
- new net SD_MOSI: J2.3 (MOSI), uC1. (TX)
- new net SD_SCK: J2.2 (SCK), uC1. (TX)
- new net S_C_DT: S2.6 (DT), uC1. (TX)
- new net S_C_OU1: U1. (VCC), uC1. (TX)
- new net S_C_SCK: S2.7 (SCK), uC1. (TX)
- new net S_I_OUT: S1. (VCC), uC1. (TX)
- no-connect marks 0 -> 1
Other:
- note added: "Alimentación"
- note added: "Interfaz con el usuario"
- note added: "Sensores"
- note added: "uC"
- moved on the sheet: C1, DS1, E1, S1, S3, U1

Commit message: Ultima version
Parts:
- added D1: 1N4752, symbol Diode:1N47xxA
- added J3: (no value), symbol Connector:Screw_Terminal_01x02
- added R3: 1M, Resistor_SMD:R_1206_3216Metric, symbol Device:R
- added R4: 100k, Resistor_SMD:R_1206_3216Metric, symbol Device:R
- C2: value (none) -> 220uF
- C4: value (none) -> 100nF; footprint (none) -> Capacitor_SMD:C_1206_3216Metric
- J2: footprint (none) -> Connector_Molex:Molex_KK-254_AE-6410-06A_1x06_P2.54mm_Vertical
- R1, R2: renamed from R?; value (none) -> 100k; footprint (none) -> Resistor_SMD:R_1206_3216Metric
- U1: footprint (none) -> Connector_Molex:Molex_KK-254_AE-6410-03A_1x03_P2.54mm_Vertical
Connections:
- net BAT+: no longer R1.1
- net BAT+_EXT: now also R3.2, R4.1
- net GND: now also D1.2 (A), R4.2
- new net BAText+: D1.1 (K), J3.2 (Pin_2), R3.1
- new net BATint+: J3.1 (Pin_1), R1.1

Commit message: <Revisión PCB y STEP>
Parts:
- D1: footprint (none) -> Diode_SMD:D_MiniMELF
- J3: value (none) -> Baterias; footprint (none) -> Connector_Molex:Molex_KK-254_AE-6410-02A_1x02_P2.54mm_Vertical
Other:
- note added: "Medición voltaje de baterias"
- moved on the sheet: C3, C4, D1, DS1, E1, J2, J3, R1, R2, R3, R4, uC1
